File: sunrise.kicad_pcb (KiCad board)
At the start: 2 copper layers, 43.4 x 25.4 mm, 16 parts, among them J1 TOP_HDR, J2 BTM_HDR, U1 LM3410, U2 LP5012

Commit message: Update RGBW footprint and BOM.
Parts:
- D2, D3, D4, D5: footprint sunrise:LED_RBGW_PLCC-8 -> sunrise:LED_SMD5050-8
- turned D2 to 180 degrees
- turned D3 to 180 degrees
- turned D4 to 0 degrees
- turned D5 to 0 degrees
Connections:
- D2 pad 1: /FB_WHT -> VCC
- D2 pad 2: /OUT2 -> VCC
- D2 pad 3: /OUT1 -> VCC
- D2 pad 4: /OUT0 -> Net-(D2-Pad4)
- D2 pad 5: VCC -> /FB_WHT
- D2 pad 6: VCC -> /OUT2
- D2 pad 7: VCC -> /OUT1
- D2 pad 8: Net-(D2-Pad8) -> /OUT0
- D3 pad 1: Net-(D2-Pad8) -> VCC
- D3 pad 2: /OUT5 -> VCC
- D3 pad 3: /OUT4 -> VCC
- D3 pad 4: /OUT3 -> Net-(D3-Pad4)
- D3 pad 5: VCC -> Net-(D2-Pad4)
- D3 pad 6: VCC -> /OUT5
- D3 pad 7: VCC -> /OUT4
- D3 pad 8: Net-(D3-Pad8) -> /OUT3
- D4 pad 1: Net-(D3-Pad8) -> VCC
- D4 pad 2: /OUT8 -> VCC
- D4 pad 3: /OUT7 -> VCC
- D4 pad 4: /OUT6 -> Net-(D4-Pad4)
- D4 pad 5: VCC -> Net-(D3-Pad4)
- D4 pad 6: VCC -> /OUT8
- D4 pad 7: VCC -> /OUT7
- D4 pad 8: Net-(D4-Pad8) -> /OUT6
- D5 pad 1: Net-(D4-Pad8) -> VCC
- D5 pad 2: /OUT11 -> VCC
- D5 pad 3: /OUT10 -> VCC
- D5 pad 4: /OUT9 -> /V_{OUT}_WHT
- D5 pad 5: VCC -> Net-(D4-Pad4)
- D5 pad 6: VCC -> /OUT11
- D5 pad 7: VCC -> /OUT10
- D5 pad 8: /V_{OUT}_WHT -> /OUT9
Routing:
- net Net-(D3-Pad4): track 0.00 -> 13.3 mm
- net Net-(D3-Pad8): track 13.1 -> 0.00 mm
- net Net-(D4-Pad8): track 2.82 -> 0.00 mm
- net Net-(D4-Pad4): track 0.00 -> 2.82 mm
- net Net-(D2-Pad8): track 2.82 -> 0.00 mm
- net Net-(D2-Pad4): track 0.00 -> 2.82 mm
- net VCC: track 9.33 -> 9.69 mm, vias 22 -> 19
Other:
- board text added: "+5V"
- board text added: "+5V GND"
- board text added: "ADDR0"
- board text added: "ADDR1"
- board text added: "EN"
- board text added: "GND"
- board text added: "PWM WHT"
- board text added: "SCL"
- board text added: "SDA"
